Commit message: 6dof_edit

File: my_robot_description/src/my_robot_description/urdf/arm.xacro (robot description, xacro)
@@ -25,4 +25,55 @@
                            xyz="0 0 ${arm_base_height / 2.0}" rpy="0 0 0" />
     </link>
+    <link name="arm_base_link2">
+        <visual>
+            <geometry>
+                <box size="${arm_base_length} ${arm_base_width} ${arm_base_height}" />
+            </geometry>
+            <origin xyz="0 0 ${arm_base_height / 2.0}" rpy="0 0 0" />
+            <material name="orange" />
+        </visual>
+        <collision>
+            <geometry>
+                <box size="${arm_base_length} ${arm_base_width} ${arm_base_height}" />
+            </geometry>
+            <origin xyz="0 0 ${arm_base_height / 2.0}" rpy="0 0 0" />
+        </collision>
+        <xacro:box_inertia m="0.03" l="${2*arm_base_length}" w="${2*arm_base_width}" h="${2*arm_base_height}"
+                           xyz="0 0 ${arm_base_height / 2.0}" rpy="0 0 0" />
+    </link>
+ <link name="arm_base_link3">
+        <visual>
+            <geometry>
+                <box size="${arm_base_length} ${arm_base_width} ${arm_base_height}" />
+            </geometry>
+            <origin xyz="0 0 ${arm_base_height / 2.0}" rpy="0 0 0" />
+            <material name="orange" />
+        </visual>
+        <collision>
+            <geometry>
+                <box size="${arm_base_length} ${arm_base_width} ${arm_base_height}" />
+            </geometry>
+            <origin xyz="0 0 ${arm_base_height / 2.0}" rpy="0 0 0" />
+        </collision>
+        <xacro:box_inertia m="0.01" l="${2*arm_base_length}" w="${2*arm_base_width}" h="${2*arm_base_height}"
+                           xyz="0 0 ${arm_base_height / 2.0}" rpy="0 0 0" />
+    </link>
+    <link name="arm_base_link4">
+        <visual>
+            <geometry>
+                <box size="${arm_base_length} ${arm_base_width} ${arm_base_height}" />
+            </geometry>
+            <origin xyz="0 0 ${arm_base_height / 2.0}" rpy="0 0 0" />
+            <material name="orange" />
+        </visual>
+        <collision>
+            <geometry>
+                <box size="${arm_base_length} ${arm_base_width} ${arm_base_height}" />
+            </geometry>
+            <origin xyz="0 0 ${arm_base_height / 2.0}" rpy="0 0 0" />
+        </collision>
+        <xacro:box_inertia m="0.01" l="${2*arm_base_length}" w="${2*arm_base_width}" h="${2*arm_base_height}"
+                           xyz="0 0 ${arm_base_height / 2.0}" rpy="0 0 0" />
+    </link>
     <link name="forearm_link">
         <visual>
@@ -39,5 +90,5 @@
             <origin xyz="0 0 ${forearm_length / 2.0}" rpy="0 0 0" />
         </collision>
-        <xacro:cylinder_inertia m="0.3" r="${2*forearm_radius}" h="${2*forearm_length}"
+        <xacro:cylinder_inertia m="0.03" r="${2*forearm_radius}" h="${2*forearm_length}"
                                 xyz="0 0 ${forearm_length / 2.0}" rpy="0 0 0" />
     </link>
@@ -56,13 +107,21 @@
             <origin xyz="0 0 ${hand_length / 2.0}" rpy="0 0 0" />
         </collision>
-        <xacro:cylinder_inertia m="0.3" r="${2*hand_radius}" h="${2*hand_length}"
+        <xacro:cylinder_inertia m="0.03" r="${2*hand_radius}" h="${2*hand_length}"
                                 xyz="0 0 ${hand_length / 2.0}" rpy="0 0 0" />
     </link>
+    <joint name="arm_base_2_joint" type="revolute">
+        <parent link="arm_base_link2" />
+        <child link="arm_base_link" />
+        <origin xyz="0 0 ${arm_base_height}" rpy="0 0 0" />
+        <axis xyz="0 0 1" />
+        <limit lower="0" upper="${pi*2}" effort="200" velocity="100" />
+        <dynamics friction="3.05" damping="1.0" />
+    </joint>
     <joint name="arm_base_forearm_joint" type="revolute">
         <parent link="arm_base_link" />
         <child link="forearm_link" />
-        <origin xyz="0 0 ${arm_base_height}" rpy="0 0 0" />
+        <origin xyz="0 0 ${arm_base_height*2}" rpy="0 0 0" />
         <axis xyz="0 1 0" />
-        <limit lower="0" upper="${pi*2}" effort="200" velocity="100" />
+        <limit lower="${-pi*2}" upper="${pi*2}" effort="200" velocity="100" />
         <dynamics friction="3.05" damping="1.0" />
     </joint>
@@ -72,4 +131,20 @@
         <origin xyz="0 0 ${forearm_length}" rpy="0 0 0" />
         <axis xyz="0 1 0" />
+        <limit lower="${-pi*2}" upper="${pi*2}" effort="200" velocity="100" />
+        <dynamics friction="3.05" damping="1.0" />
+    </joint>
+    <joint name="hand_2_joint" type="revolute">
+        <parent link="hand_link" />
+        <child link="arm_base_link3" />
+        <origin xyz="0 0 ${hand_length}" rpy="0 0 0" />
+        <axis xyz="0 0 1" />
+        <limit lower="0" upper="${pi*2}" effort="200" velocity="100" />
+        <dynamics friction="3.05" damping="1.0" />
+    </joint>
+    <joint name="hand_3_joint" type="revolute">
+        <parent link="arm_base_link3" />
+        <child link="arm_base_link4" />
+        <origin xyz="0 0 0.09" rpy="0 0 0" />
+        <axis xyz="1 0 0" />
         <limit lower="0" upper="${pi*2}" effort="200" velocity="100" />
         <dynamics friction="3.05" damping="1.0" />

File: my_robot_description/src/my_robot_description/urdf/arm_gazebo.xacro (robot description, xacro)
@@ -17,5 +17,8 @@
             <!-- Name of joints in the model whose states will be published. -->
             <joint_name>arm_base_forearm_joint</joint_name>
+            <joint_name>arm_base_2_joint</joint_name>
             <joint_name>forearm_hand_joint</joint_name>
+            <joint_name>hand_2_joint</joint_name>
+            <joint_name>hand_3_joint</joint_name>
             <joint_name>base_camera_joint</joint_name>
         </plugin>

File: my_robot_description/src/my_robot_description/urdf/camera.xacro (robot description, xacro)
@@ -20,7 +20,7 @@
      </link>
      <joint name="base_camera_joint" type="revolute">
-         <parent link="hand_link"/>
+         <parent link="arm_base_link4"/>
          <child link="camera_link" />
-         <origin xyz="0 0 0.6 " rpy="0 ${pi*2} 0" />
+         <origin xyz="0 0 0.07 " rpy="0 ${pi*2} 0" />
          <axis xyz="0 -1 0" />
         <limit lower="0" upper="${pi*2}" effort="200" velocity="100" />

File: my_robot_description/src/my_robot_description/urdf/my_robot.urdf.xacro (robot description, xacro)
@@ -9,4 +9,5 @@
     <xacro:include filename="lidar.xacro" />
     <xacro:include filename="lidar2.xacro" />
+    <xacro:include filename="lidar3.xacro" />
     <!-- <xacro:include filename="dokari.xacro" />
     <xacro:include filename="camera3_dokari.xacro" />
@@ -21,5 +22,5 @@
     <joint name="mobilebasearm_joint" type="fixed">
          <parent link="base_link"/>
-         <child link="arm_base_link" />
+         <child link="arm_base_link2" />
          <origin xyz="0.2 0 ${base_height + 0.01}" rpy="0 0 ${pi / 2.0} " />
      </joint>
